Commit message: Corrected for lidar +y direction

File: packages/orbirob_description/urdf/OrbiRob.urdf (robot description, URDF)
Before this commit: robot OrbiRob, 5 links, 4 joints
Joints:
- joint lidar_joint: origin xyz=0.00829037 0.0 0.293108 rpy=3.141592653589793 0.026179938779890263 3.141592653589793 -> xyz=0.00829037 0.0 0.293108 rpy=0 0.026179938779890263 3.141592653589793

Commit message: revised for gazebo

File: packages/orbirob_description/urdf/OrbiRob.urdf (robot description, URDF)
Before this commit: robot OrbiRob, 5 links, 4 joints
Joints:
- joint wheel_left_joint: axis 0 0 1 -> 0 1 0; limit effort=0.0 velocity=0.0 -> effort=10.0 velocity=10.0
- joint wheel_right_joint: axis 0 0 1 -> 0 1 0; limit effort=0.0 velocity=0.0 -> effort=10.0 velocity=10.0

Commit message: revised for gazebo

File: packages/orbirob_description/urdf/OrbiRob.urdf (robot description, URDF)
Before this commit: robot OrbiRob, 5 links, 4 joints
Links:
- added link caster_front_link, mass 0.025; collision cylinder length=0.01 radius=0.012; visual mesh filename=package://orbirob_description/meshes/bearings.dae
- added link caster_rear_link, mass 0.025; collision cylinder length=0.01 radius=0.012; visual mesh filename=package://orbirob_description/meshes/bearings.dae
- link base_link: geometry collision cylinder length=0.38885000000000003 radius=0.2399906471807673; visual mesh filename=package://orbirob_description/meshes/boardhwor001.dae
- link wheel_left_link: geometry collision cylinder length=0.03 radius=0.04; visual mesh filename=package://orbirob_description/meshes/wheel_left_link_.dae
- link wheel_right_link: geometry collision cylinder length=0.03 radius=0.04; visual mesh filename=package://orbirob_description/meshes/wheel_right_link_.dae
Joints:
- added joint caster_front_joint: type fixed, parent base_link, child caster_front_link, origin xyz=0.0 0.0 0.0 rpy=0 0 0
- added joint caster_rear_joint: type fixed, parent caster_rear_link, child base_link, origin xyz=0.0 0.0 0.0 rpy=0 0 0
- joint lidar_joint: origin xyz=0.00829037 0.0 0.293108 rpy=0 0.026179938779890263 3.141592653589793 -> xyz=0.00829037 0.0 0.293108 rpy=0 0.026179938779890274 3.141592653589793
- joint wheel_left_joint: axis 0 1 0 -> 0 0 -1; limit effort=10.0 velocity=10.0 -> effort=0.0 velocity=0.0; origin xyz=0.0 0.1631 0.03915 rpy=0 -1.332800375e-07 0 -> xyz=0.0 0.1481 0.03915 rpy=-1.5707963267948966 -2.564103401974412e-08 3.141592653589793
- joint wheel_right_joint: axis 0 1 0 -> 0 0 -1; limit effort=10.0 velocity=10.0 -> effort=0.0 velocity=0.0; origin xyz=0.0 -0.1522 0.03915 rpy=0 0 0 -> xyz=0.0 -0.1482 0.03915 rpy=-1.5707963267948968 0 -3.141592653589793
